File: Procab 700 Sim/Class700Sim/Class700Sim.kicad_sch (KiCad schematic)
At the start: 90 parts

Commit message: Drew Main Driving Panel
Parts:
- added D1: LED-DLL, symbol Device:LED
- added D2: LED-DLR, symbol Device:LED
- added D3: LED-SND, symbol Device:LED
- added J1: DB25 Male Connector, Connector_Dsub:DSUB-25_Pins_Vertical_P2.77x2.84mm, symbol Connector:DB25_Pins
- added J2: DB25 Female Connector, Connector_Dsub:DSUB-25_Pins_Vertical_P2.77x2.84mm, symbol Connector:DB25_Socket
- added SW1: SW-DPTTN, symbol Switch:SW_SPST
- added SW10: SW-DRR1, symbol Switch:SW_SPST
- added SW11: SW-DRR2, symbol Switch:SW_SPST
- added SW12: SW-DCR, symbol Switch:SW_SPST
- added SW13: SW-HRNH, symbol Switch:SW_SPST
- added SW14: SW-HRNL, symbol Switch:SW_SPST
- added SW15: SW-SND, symbol Switch:SW_SPST
- added SW16: SW-ATSP, symbol Switch:SW_SPST
- added SW17: SW-ATSA, symbol Switch:SW_SPST
- added SW18: SW-ETA, symbol Switch:SW_SPST
- added SW19: SW-AWS, symbol Switch:SW_SPST
- added SW2: SW-DRL1, symbol Switch:SW_SPST
- added SW3: SW-DRL2, symbol Switch:SW_SPST
- added SW4: SW-DCL, symbol Switch:SW_SPST
- added SW5: SW-SB, symbol Switch:SW_SPST
- added SW6: SW-MK, symbol Switch:SW_SPST
- added SW7: SW-REVF, symbol Switch:SW_SPST
- added SW8: SW-REVR, symbol Switch:SW_SPST
Connections:
- net DI1: now also D1.1 (K), D2.1 (K), J1.14 (P14), J1.24 (P24), J1.3, J2.14 (P14), J2.24 (P24), J2.3, SW1. (B)
- net DI10: now also J1.21 (P21), J2.21 (P21), SW17. (B)
- net DI11: now also J1.9, J2.9, SW16. (B)
- net DI12: now also J1.10, J2.10, SW15. (B)
- net DI13: now also J1.23 (P23), J2.23 (P23), SW14. (B)
- net DI14: now also J1.11, J2.11, SW13. (B)
- net DI15: now also J1.12, J2.12, SW12. (B)
- net DI16: now also J1.25 (P25), J2.25 (P25), SW10. (B)
- net DI2: now also D3.1 (K), J1.2, J1.22 (P22), J2.2, J2.22 (P22), SW2. (B)
- net DI3: now also J1.15 (P15), J2.15 (P15), SW4. (B)
- net DI4: now also J1.16 (P16), J2.16 (P16), SW5. (B)
- net DI5: now also J1.4, J2.4, SW6. (B)
- net DI6: now also J1.17 (P17), J2.17 (P17), SW7. (B)
- net DI7: now also J1.5, J2.5, SW8. (B)
- net DI8: now also J1.20 (P20), J2.20 (P20), SW19. (B)
- net DI9: now also J1.8, J2.8, SW18. (B)
- new net PA2000: D1.2 (A), J1.13, J2.13, SW1. (B), SW3. (B), SW4. (B), SW5. (B), SW6. (B), SW7. (B), SW8. (B)
- new net PA2010: SW2. (B), SW3. (B)
- new net PA4000: D2.2 (A), D3.2 (A), J1.1, J2.1, SW11. (B), SW12. (B), SW13. (B), SW14. (B), SW15. (B), SW16. (B), SW17. (B), SW18. (B), SW19. (B)
- new net PA4010: SW10. (B), SW11. (B)
- no-connect marks 0 -> 8
Other:
- added sheet Brake Gauge Panel (Brake Gauge Panel.kicad_sch)
- note added: "40 39 38 37 36 35 34 33 32 31 30 29 28 27 26 25 24 23 22 21 20 19 18 17 16 15 14 13 12 11 10 9 8 7 6 5 4 3 2 1"
- note added: "90 89 88 87 86 85 84 83 82 81 80 79 78 77 76 75 74 73 72 71 70 69 68 67 66 65 64 63 62 61 60 59 58 57 56 55 54 53 52 51 50 49 48 47 46 45 44 43 42 41"
- note added: "DB25 Female Connector Connections"
- note added: "DB25 Male Connector"
- note added: "DB25 Male Connector Connections"
- note added: "Main Driving Panel"
- note removed: "1 2 3 4 5 6 7 8 9 10 11 12 13 14 15 16 17 18 19 20 21 22 23 24 25 26 27 28 29 30 31 32 33 34 35 36 37 38 39 40"
- note removed: "41 42 43 44 45 46 47 48 49 50 51 52 53 54 55 56 57 58 59 60 61 62 63 64 65 66 67 68 69 70 71 72 73 74 75 76 77 78 79 80 81 82 83 84 85 86 87 88 89 90"
- title: (none) -> Class 700 Compact Simulator Electrical

Commit message: Drew the air gauge panel
Parts:
- removed SW7: SW-REVF, symbol Switch:SW_SPST
- removed SW8: SW-REVR, symbol Switch:SW_SPST
- added SW20: SW-HRNL, symbol Switch:SW_SPST
- added SW21: SW-HRNH, symbol Switch:SW_SPST
Connections:
- net DI13: no longer SW14. (B)
- net DI14: no longer SW13. (B)
- net PA2000: now also J1.1, J2.1; no longer J1.13, J2.13
- net PA4000: now also J1.13, J2.13, SW20. (B), SW21. (B); no longer J1.1, J2.1
Other:
- note added: "SW-FNR"
- note added: "SW-HRN"

Commit message: Changes made
Other:
- note added: "Air Gauge Panel"

Commit message: TB2 added
Parts:
- added B91, B92, B93: ~, symbol DinRailTB:Din_Terminal_Blockx2_Red
- added B94, B95, B96: ~, symbol DinRailTB:Din_Terminal_Blockx2_Blue
Other:
- note added: "1 2 3 4 5 6 7 8 9 10 11 12 13 14 15 16 17 18 19 20 21 22 23 24 25 26 27 28 29 30 31 32 33 34 35 36 37 38 39 40"
- note added: "41 42 43 44 45 46 47 48 49 50 51 52 53 54 55 56 57 58 59 60 61 62 63 64 65 66 67 68 69 70 71 72 73 74 75 76 77 78 79 80 81 82 83 84 85 86 87 88 89 90"
- note added: "TB2"
- note added: "To Air Gauge Panel"
- note removed: "40 39 38 37 36 35 34 33 32 31 30 29 28 27 26 25 24 23 22 21 20 19 18 17 16 15 14 13 12 11 10 9 8 7 6 5 4 3 2 1"
- note removed: "90 89 88 87 86 85 84 83 82 81 80 79 78 77 76 75 74 73 72 71 70 69 68 67 66 65 64 63 62 61 60 59 58 57 56 55 54 53 52 51 50 49 48 47 46 45 44 43 42 41"
